Commit message: added floor joint to URDF

File: pi/src/urdf/src/DCMR-4W01.urdf (robot description, URDF)
Before this commit: robot DCMR-4W01, 6 links, 5 joints
Links:
- added link base_footprint
Joints:
- added joint floor_joint: type fixed, parent base_footprint, child base_link, origin xyz=0 0 0.025 rpy=0 0 0
